Commit message: Update igus_rebel_moveit_config package
- Improve Igus Rebel URDF (remove gaps, use actual geometry from CAD file)
- Remove unused interfaces
- Remove control aspects from Igus Rebel description package, isolate to moveit config package

File: igus_rebel_description/urdf/Rebel.xacro (robot description, xacro)
@@ -148,5 +148,5 @@
   <parent link="base_link"/>
   <child link="link_1_1"/>
-  <axis xyz="-0.0 0.0 -1.0"/>
+  <axis xyz="0.0 0.0 1.0"/>
   <limit upper="3.124139" lower="-3.124139" effort="100" velocity="100"/>
 </joint>
@@ -169,5 +169,5 @@
   <parent link="link_3_1"/>
   <child link="link_4_1"/>
-  <axis xyz="0.0 9e-06 -1.0"/>
+  <axis xyz="0.0 0.0 1.0"/>
   <limit upper="3.124139" lower="-3.124139" effort="100" velocity="100"/>
 </joint>
@@ -176,5 +176,5 @@
   <parent link="link_4_1"/>
   <child link="link_5_1"/>
-  <axis xyz="-1.0 -0.0 -0.0"/>
+  <axis xyz="1.0 0.0 -0.0"/>
   <limit upper="1.658063" lower="-1.658063" effort="100" velocity="100"/>
 </joint>
@@ -183,5 +183,5 @@
   <parent link="link_5_1"/>
   <child link="link_eef_1"/>
-  <axis xyz="-0.0 -1e-05 1.0"/>
+  <axis xyz="-0.0 0.0 1.0"/>
   <limit upper="3.124139" lower="-3.124139" effort="100" velocity="100"/>
 </joint>

Commit message: Update base_link to link_base
- Changed to avoid conflicts when integrating with woody

File: igus_rebel_description/urdf/Rebel.xacro (robot description, xacro)
@@ -4,5 +4,5 @@
 <xacro:include filename="$(find igus_rebel_description)/urdf/Rebel.trans" />
 <xacro:include filename="$(find igus_rebel_description)/urdf/Rebel.gazebo" />
-<link name="base_link">
+<link name="link_base">
   <inertial>
     <origin xyz="0.0002483693748801606 -0.0012903342275887133 0.03950362292761386" rpy="0 0 0"/>
@@ -146,5 +146,5 @@
 <joint name="joint1" type="revolute">
   <origin xyz="0.0 0.0 0.1" rpy="0 0 0"/>
-  <parent link="base_link"/>
+  <parent link="link_base"/>
   <child link="link_1_1"/>
   <axis xyz="0.0 0.0 1.0"/>

Commit message: Change link_eef name

File: igus_rebel_description/urdf/Rebel.xacro (robot description, xacro)
@@ -124,5 +124,5 @@
   </collision>
 </link>
-<link name="link_eef_1">
+<link name="link_eef">
   <inertial>
     <origin xyz="-1.749470192662973e-13 -0.00029348300701733667 -0.0007690227381885739" rpy="0 0 0"/>
@@ -182,5 +182,5 @@
   <origin xyz="0.033 0.000482 0.1273" rpy="0 0 0"/>
   <parent link="link_5_1"/>
-  <child link="link_eef_1"/>
+  <child link="link_eef"/>
   <axis xyz="-0.0 0.0 1.0"/>
   <limit upper="3.124139" lower="-3.124139" effort="100" velocity="100"/>
